Commit message: Make the priliminary urdf model. collision present among joints

File: install/rrbot_description/share/rrbot_description/urdf/rrbot_description.urdf.xacro (robot description, xacro)
@@ -1,112 +1,147 @@
 <?xml version="1.0"?>
 <robot xmlns:xacro="http://www.ros.org/wiki/xacro">
+  <!-- Launch RVIZ using ros2 launch rrbot_description view_robot.launch.py -->
   <xacro:macro name="rrbot" params="parent prefix *origin">
-  <!-- Constants for robot dimensions -->
-  <xacro:property name="mass" value="1" /> <!-- arbitrary value for mass -->
-  <xacro:property name="width" value="0.1" /> <!-- Square dimensions (widthxwidth) of beams -->
-  <xacro:property name="height1" value="2" /> <!-- Link 1 -->
-  <xacro:property name="height2" value="1" /> <!-- Link 2 -->
-  <xacro:property name="height3" value="1" /> <!-- Link 3 -->
-  <xacro:property name="camera_link" value="0.05" /> <!-- Size of square 'camera' box -->
-  <xacro:property name="axel_offset" value="0.05" /> <!-- Space btw top of beam and the each joint -->
-  <joint name="${prefix}base_joint" type="fixed">
-    <xacro:insert_block name="origin" />
-    <parent link="${parent}"/>
-    <child link="${prefix}base_link" />
-  </joint>
-  <!-- Base Link -->
-  <link name="${prefix}base_link">
-    <collision>
-      <origin xyz="0 0 ${height1/2}" rpy="0 0 0"/>
-      <geometry>
-        <box size="${width} ${width} ${height1}"/>
-      </geometry>
-    </collision>
-    <visual>
-      <origin xyz="0 0 ${height1/2}" rpy="0 0 0"/>
-      <geometry>
-        <box size="${width} ${width} ${height1}"/>
-      </geometry>
-      <material name="orange"/>
-    </visual>
-    <inertial>
-      <origin xyz="0 0 ${height1/2}" rpy="0 0 0"/>
-      <mass value="${mass}"/>
-      <inertia
-        ixx="${mass / 12.0 * (width*width + height1*height1)}" ixy="0.0" ixz="0.0"
-        iyy="${mass / 12.0 * (height1*height1 + width*width)}" iyz="0.0"
-        izz="${mass / 12.0 * (width*width + width*width)}"/>
-      </inertial>
-    </link>
-    <joint name="${prefix}joint1" type="continuous">
-      <parent link="${prefix}base_link"/>
-      <child link="${prefix}link1"/>
-      <origin xyz="0 ${width} ${height1 - axel_offset}" rpy="0 1.5708 0"/>
-      <axis xyz="1 0 0"/>
-      <dynamics damping="0.7"/>
+    <!-- Constants for robot dimensions -->
+    <xacro:property name="mass" value="1" />
+    <!-- arbitrary value for mass -->
+    <xacro:property name="width" value="0.1" />
+    <!-- Square dimensions (widthxwidth) of beams -->
+    <xacro:property name="base_link_length" value="1" />
+    <!-- Link 1 -->
+    <xacro:property name="link1_length" value="1" />
+    <!-- Link 2 -->
+    <xacro:property name="link2_length" value="1" />
+    <!-- Link 3 -->
+    <xacro:property name="link3_length" value="1" />
+    <!-- Link 4 -->
+    <xacro:property name="camera_link" value="0.05" />
+    <!-- Size of square 'camera' box -->
+    <xacro:property name="axel_offset" value="0.05" />
+    <!-- Space btw top of beam and the each joint -->
+    <!-- Joint 0: Fixed -->
+    <joint name="${prefix}base_joint" type="fixed">
+      <xacro:insert_block name="origin" />
+      <parent link="${parent}"/>
+      <child link="${prefix}base_link" />
     </joint>
-    <!-- Middle Link -->
-    <link name="${prefix}link1">
+    <!-- Base Link -->
+    <link name="${prefix}base_link">
       <collision>
-        <origin xyz="0 0 ${height2/2 - axel_offset}" rpy="0 0 0"/>
+        <origin xyz="0 0 ${base_link_length/2}" rpy="0 0 0"/>
         <geometry>
-          <box size="${width} ${width} ${height2}"/>
+          <box size="${width} ${width} ${base_link_length}"/>
         </geometry>
       </collision>
       <visual>
-        <origin xyz="0 0 ${height2/2 - axel_offset}" rpy="0 0 0"/>
+        <origin xyz="0 0 ${base_link_length/2}" rpy="0 0 0"/>
         <geometry>
-          <box size="${width} ${width} ${height2}"/>
+          <box size="${width} ${width} ${base_link_length}"/>
         </geometry>
         <material name="yellow"/>
       </visual>
       <inertial>
-        <origin xyz="0 0 ${height2/2 - axel_offset}" rpy="0 0 0"/>
+        <origin xyz="0 0 ${base_link_length/2}" rpy="0 0 0"/>
         <mass value="${mass}"/>
-        <inertia
-          ixx="${mass / 12.0 * (width*width + height2*height2)}" ixy="0.0" ixz="0.0"
-          iyy="${mass / 12.0 * (height2*height2 + width*width)}" iyz="0.0"
-          izz="${mass / 12.0 * (width*width + width*width)}"/>
-        </inertial>
-      </link>
-      <joint name="${prefix}joint2" type="continuous">
-        <parent link="${prefix}link1"/>
-        <child link="${prefix}link2"/>
-        <origin xyz="0 ${width} ${height2 - axel_offset*2}" rpy="0 0 0"/>
-        <axis xyz="1 0 0"/>
-        <dynamics damping="0.7"/>
-      </joint>
-      <!-- Top Link -->
-      <link name="${prefix}link2">
-        <collision>
-          <origin xyz="0 0 ${height3/2 - axel_offset}" rpy="0 0 0"/>
-          <geometry>
-            <box size="${width} ${width} ${height3}"/>
-          </geometry>
-        </collision>
-        <visual>
-          <origin xyz="0 0 ${height3/2 - axel_offset}" rpy="0 0 0"/>
-          <geometry>
-            <box size="${width} ${width} ${height3}"/>
-          </geometry>
-          <material name="orange"/>
-        </visual>
-        <inertial>
-          <origin xyz="0 0 ${height3/2 - axel_offset}" rpy="0 0 0"/>
-          <mass value="${mass}"/>
-          <inertia
-            ixx="${mass / 12.0 * (width*width + height3*height3)}" ixy="0.0" ixz="0.0"
-            iyy="${mass / 12.0 * (height3*height3 + width*width)}" iyz="0.0"
-            izz="${mass / 12.0 * (width*width + width*width)}"/>
-          </inertial>
-        </link>
-        <joint name="${prefix}tool_joint" type="fixed">
-          <origin xyz="0 0 1" rpy="0 0 0" />
-          <parent link="${prefix}link2"/>
-          <child link="${prefix}tool_link" />
-        </joint>
-        <!-- Tool Link -->
-        <link name="${prefix}tool_link">
-        </link>
+        <inertia ixx="${mass / 12.0 * (width*width + base_link_length*base_link_length)}" ixy="0.0" ixz="0.0" iyy="${mass / 12.0 * (base_link_length*base_link_length + width*width)}" iyz="0.0" izz="${mass / 12.0 * (width*width + width*width)}"/>
+      </inertial>
+    </link>
+    <!-- Joint 1: Revolute -->
+    <joint name="${prefix}joint1" type="continuous">
+      <parent link="${prefix}base_link"/>
+      <child link="${prefix}link1"/>
+      <origin xyz="0 0 ${base_link_length}" rpy="0 0 0"/>
+      <axis xyz="0 0 1"/>
+      <dynamics damping="0.7"/>
+    </joint>
+    <!-- Link 1 -->
+    <link name="${prefix}link1">
+      <collision>
+        <origin xyz="0 0 ${link1_length/2 - axel_offset}" rpy="0 0 0"/>
+        <geometry>
+          <box size="${width} ${width} ${link1_length}"/>
+        </geometry>
+      </collision>
+      <visual>
+        <origin xyz="0 0 ${link1_length/2 - axel_offset}" rpy="0 0 0"/>
+        <geometry>
+          <box size="${width} ${width} ${link1_length}"/>
+        </geometry>
+        <material name="orange"/>
+      </visual>
+      <inertial>
+        <origin xyz="0 0 ${link1_length/2 - axel_offset}" rpy="0 0 0"/>
+        <mass value="${mass}"/>
+        <inertia ixx="${mass / 12.0 * (width*width + link1_length*link1_length)}" ixy="0.0" ixz="0.0" iyy="${mass / 12.0 * (link1_length*link1_length + width*width)}" iyz="0.0" izz="${mass / 12.0 * (width*width + width*width)}"/>
+      </inertial>
+    </link>
+    <!-- Joint 2: Revolute -->
+    <joint name="${prefix}joint2" type="continuous">
+      <parent link="${prefix}link1"/>
+      <child link="${prefix}link2"/>
+      <origin xyz="0 ${width} ${link1_length - axel_offset*2}" rpy="0 0 0"/>
+      <axis xyz="1 0 0"/>
+      <dynamics damping="0.7"/>
+    </joint>
+    <!-- Link 2 -->
+    <link name="${prefix}link2">
+      <collision>
+        <origin xyz="0 0 ${link2_length/2 - axel_offset}" rpy="0 0 0"/>
+        <geometry>
+          <box size="${width} ${width} ${link2_length}"/>
+        </geometry>
+      </collision>
+      <visual>
+        <origin xyz="0 0 ${link2_length/2 - axel_offset}" rpy="0 0 0"/>
+        <geometry>
+          <box size="${width} ${width} ${link2_length}"/>
+        </geometry>
+        <material name="orange"/>
+      </visual>
+      <inertial>
+        <origin xyz="0 0 ${link2_length/2 - axel_offset}" rpy="0 0 0"/>
+        <mass value="${mass}"/>
+        <inertia ixx="${mass / 12.0 * (width*width + link2_length*link2_length)}" ixy="0.0" ixz="0.0" iyy="${mass / 12.0 * (link2_length*link2_length + width*width)}" iyz="0.0" izz="${mass / 12.0 * (width*width + width*width)}"/>
+      </inertial>
+    </link>
+    <!-- Joint 3: Prismatic -->
+    <joint name="${prefix}joint3" type="prismatic">
+      <limit effort="50" lower="0" upper="${link3_length - 2*axel_offset}" velocity="10"/>
+      <parent link="${prefix}link2"/>
+      <child link="${prefix}link3"/>
+      <origin xyz="0 ${width} ${link2_length - axel_offset*2}" rpy="0 1.5703 0"/>
+      <axis xyz="0 0 -1"/>
+      <dynamics damping="0.7"/>
+    </joint>
+    <!-- Link 3 -->
+    <link name="${prefix}link3">
+      <collision>
+        <origin xyz="0 0 ${link3_length/2 - axel_offset}" rpy="0 0 0"/>
+        <geometry>
+          <box size="${width} ${width} ${link3_length}"/>
+        </geometry>
+      </collision>
+      <visual>
+        <origin xyz="0 0 ${link3_length/2 - axel_offset}" rpy="0 0 0"/>
+        <geometry>
+          <box size="${width} ${width} ${link3_length}"/>
+        </geometry>
+        <material name="orange"/>
+      </visual>
+      <inertial>
+        <origin xyz="0 0 ${link3_length/2 - axel_offset}" rpy="0 0 0"/>
+        <mass value="${mass}"/>
+        <inertia ixx="${mass / 12.0 * (width*width + link3_length*link3_length)}" ixy="0.0" ixz="0.0" iyy="${mass / 12.0 * (link3_length*link3_length + width*width)}" iyz="0.0" izz="${mass / 12.0 * (width*width + width*width)}"/>
+      </inertial>
+    </link>
+    <!-- Tool Joint: Virtual -->
+    <joint name="${prefix}tool_joint" type="fixed">
+      <origin xyz="0 0 1" rpy="0 0 0" />
+      <parent link="${prefix}link3"/>
+      <child link="${prefix}tool_link" />
+    </joint>
+    <!-- Tool Link -->
+    <link name="${prefix}tool_link">
+    </link>
   </xacro:macro>
 </robot>

File: src/rrbot_simulation_files/rrbot_description/urdf/rrbot_description.urdf.xacro (robot description, xacro)
@@ -1,112 +1,147 @@
 <?xml version="1.0"?>
 <robot xmlns:xacro="http://www.ros.org/wiki/xacro">
+  <!-- Launch RVIZ using ros2 launch rrbot_description view_robot.launch.py -->
   <xacro:macro name="rrbot" params="parent prefix *origin">
-  <!-- Constants for robot dimensions -->
-  <xacro:property name="mass" value="1" /> <!-- arbitrary value for mass -->
-  <xacro:property name="width" value="0.1" /> <!-- Square dimensions (widthxwidth) of beams -->
-  <xacro:property name="height1" value="2" /> <!-- Link 1 -->
-  <xacro:property name="height2" value="1" /> <!-- Link 2 -->
-  <xacro:property name="height3" value="1" /> <!-- Link 3 -->
-  <xacro:property name="camera_link" value="0.05" /> <!-- Size of square 'camera' box -->
-  <xacro:property name="axel_offset" value="0.05" /> <!-- Space btw top of beam and the each joint -->
-  <joint name="${prefix}base_joint" type="fixed">
-    <xacro:insert_block name="origin" />
-    <parent link="${parent}"/>
-    <child link="${prefix}base_link" />
-  </joint>
-  <!-- Base Link -->
-  <link name="${prefix}base_link">
-    <collision>
-      <origin xyz="0 0 ${height1/2}" rpy="0 0 0"/>
-      <geometry>
-        <box size="${width} ${width} ${height1}"/>
-      </geometry>
-    </collision>
-    <visual>
-      <origin xyz="0 0 ${height1/2}" rpy="0 0 0"/>
-      <geometry>
-        <box size="${width} ${width} ${height1}"/>
-      </geometry>
-      <material name="orange"/>
-    </visual>
-    <inertial>
-      <origin xyz="0 0 ${height1/2}" rpy="0 0 0"/>
-      <mass value="${mass}"/>
-      <inertia
-        ixx="${mass / 12.0 * (width*width + height1*height1)}" ixy="0.0" ixz="0.0"
-        iyy="${mass / 12.0 * (height1*height1 + width*width)}" iyz="0.0"
-        izz="${mass / 12.0 * (width*width + width*width)}"/>
-      </inertial>
-    </link>
-    <joint name="${prefix}joint1" type="continuous">
-      <parent link="${prefix}base_link"/>
-      <child link="${prefix}link1"/>
-      <origin xyz="0 ${width} ${height1 - axel_offset}" rpy="0 1.5708 0"/>
-      <axis xyz="1 0 0"/>
-      <dynamics damping="0.7"/>
+    <!-- Constants for robot dimensions -->
+    <xacro:property name="mass" value="1" />
+    <!-- arbitrary value for mass -->
+    <xacro:property name="width" value="0.1" />
+    <!-- Square dimensions (widthxwidth) of beams -->
+    <xacro:property name="base_link_length" value="1" />
+    <!-- Link 1 -->
+    <xacro:property name="link1_length" value="1" />
+    <!-- Link 2 -->
+    <xacro:property name="link2_length" value="1" />
+    <!-- Link 3 -->
+    <xacro:property name="link3_length" value="1" />
+    <!-- Link 4 -->
+    <xacro:property name="camera_link" value="0.05" />
+    <!-- Size of square 'camera' box -->
+    <xacro:property name="axel_offset" value="0.05" />
+    <!-- Space btw top of beam and the each joint -->
+    <!-- Joint 0: Fixed -->
+    <joint name="${prefix}base_joint" type="fixed">
+      <xacro:insert_block name="origin" />
+      <parent link="${parent}"/>
+      <child link="${prefix}base_link" />
     </joint>
-    <!-- Middle Link -->
-    <link name="${prefix}link1">
+    <!-- Base Link -->
+    <link name="${prefix}base_link">
       <collision>
-        <origin xyz="0 0 ${height2/2 - axel_offset}" rpy="0 0 0"/>
+        <origin xyz="0 0 ${base_link_length/2}" rpy="0 0 0"/>
         <geometry>
-          <box size="${width} ${width} ${height2}"/>
+          <box size="${width} ${width} ${base_link_length}"/>
         </geometry>
       </collision>
       <visual>
-        <origin xyz="0 0 ${height2/2 - axel_offset}" rpy="0 0 0"/>
+        <origin xyz="0 0 ${base_link_length/2}" rpy="0 0 0"/>
         <geometry>
-          <box size="${width} ${width} ${height2}"/>
+          <box size="${width} ${width} ${base_link_length}"/>
         </geometry>
         <material name="yellow"/>
       </visual>
       <inertial>
-        <origin xyz="0 0 ${height2/2 - axel_offset}" rpy="0 0 0"/>
+        <origin xyz="0 0 ${base_link_length/2}" rpy="0 0 0"/>
         <mass value="${mass}"/>
-        <inertia
-          ixx="${mass / 12.0 * (width*width + height2*height2)}" ixy="0.0" ixz="0.0"
-          iyy="${mass / 12.0 * (height2*height2 + width*width)}" iyz="0.0"
-          izz="${mass / 12.0 * (width*width + width*width)}"/>
-        </inertial>
-      </link>
-      <joint name="${prefix}joint2" type="continuous">
-        <parent link="${prefix}link1"/>
-        <child link="${prefix}link2"/>
-        <origin xyz="0 ${width} ${height2 - axel_offset*2}" rpy="0 0 0"/>
-        <axis xyz="1 0 0"/>
-        <dynamics damping="0.7"/>
-      </joint>
-      <!-- Top Link -->
-      <link name="${prefix}link2">
-        <collision>
-          <origin xyz="0 0 ${height3/2 - axel_offset}" rpy="0 0 0"/>
-          <geometry>
-            <box size="${width} ${width} ${height3}"/>
-          </geometry>
-        </collision>
-        <visual>
-          <origin xyz="0 0 ${height3/2 - axel_offset}" rpy="0 0 0"/>
-          <geometry>
-            <box size="${width} ${width} ${height3}"/>
-          </geometry>
-          <material name="orange"/>
-        </visual>
-        <inertial>
-          <origin xyz="0 0 ${height3/2 - axel_offset}" rpy="0 0 0"/>
-          <mass value="${mass}"/>
-          <inertia
-            ixx="${mass / 12.0 * (width*width + height3*height3)}" ixy="0.0" ixz="0.0"
-            iyy="${mass / 12.0 * (height3*height3 + width*width)}" iyz="0.0"
-            izz="${mass / 12.0 * (width*width + width*width)}"/>
-          </inertial>
-        </link>
-        <joint name="${prefix}tool_joint" type="fixed">
-          <origin xyz="0 0 1" rpy="0 0 0" />
-          <parent link="${prefix}link2"/>
-          <child link="${prefix}tool_link" />
-        </joint>
-        <!-- Tool Link -->
-        <link name="${prefix}tool_link">
-        </link>
+        <inertia ixx="${mass / 12.0 * (width*width + base_link_length*base_link_length)}" ixy="0.0" ixz="0.0" iyy="${mass / 12.0 * (base_link_length*base_link_length + width*width)}" iyz="0.0" izz="${mass / 12.0 * (width*width + width*width)}"/>
+      </inertial>
+    </link>
+    <!-- Joint 1: Revolute -->
+    <joint name="${prefix}joint1" type="continuous">
+      <parent link="${prefix}base_link"/>
+      <child link="${prefix}link1"/>
+      <origin xyz="0 ${width} ${base_link_length - axel_offset}" rpy="0 1.5708 0"/>
+      <axis xyz="1 0 0"/>
+      <dynamics damping="0.7"/>
+    </joint>
+    <!-- Link 1 -->
+    <link name="${prefix}link1">
+      <collision>
+        <origin xyz="0 0 ${link1_length/2 - axel_offset}" rpy="0 0 0"/>
+        <geometry>
+          <box size="${width} ${width} ${link1_length}"/>
+        </geometry>
+      </collision>
+      <visual>
+        <origin xyz="0 0 ${link1_length/2 - axel_offset}" rpy="0 0 0"/>
+        <geometry>
+          <box size="${width} ${width} ${link1_length}"/>
+        </geometry>
+        <material name="orange"/>
+      </visual>
+      <inertial>
+        <origin xyz="0 0 ${link1_length/2 - axel_offset}" rpy="0 0 0"/>
+        <mass value="${mass}"/>
+        <inertia ixx="${mass / 12.0 * (width*width + link1_length*link1_length)}" ixy="0.0" ixz="0.0" iyy="${mass / 12.0 * (link1_length*link1_length + width*width)}" iyz="0.0" izz="${mass / 12.0 * (width*width + width*width)}"/>
+      </inertial>
+    </link>
+    <!-- Joint 2: Revolute -->
+    <joint name="${prefix}joint2" type="continuous">
+      <parent link="${prefix}link1"/>
+      <child link="${prefix}link2"/>
+      <origin xyz="0 ${width} ${link1_length - axel_offset*2}" rpy="0 0 0"/>
+      <axis xyz="1 0 0"/>
+      <dynamics damping="0.7"/>
+    </joint>
+    <!-- Link 2 -->
+    <link name="${prefix}link2">
+      <collision>
+        <origin xyz="0 0 ${link2_length/2 - axel_offset}" rpy="0 0 0"/>
+        <geometry>
+          <box size="${width} ${width} ${link2_length}"/>
+        </geometry>
+      </collision>
+      <visual>
+        <origin xyz="0 0 ${link2_length/2 - axel_offset}" rpy="0 0 0"/>
+        <geometry>
+          <box size="${width} ${width} ${link2_length}"/>
+        </geometry>
+        <material name="orange"/>
+      </visual>
+      <inertial>
+        <origin xyz="0 0 ${link2_length/2 - axel_offset}" rpy="0 0 0"/>
+        <mass value="${mass}"/>
+        <inertia ixx="${mass / 12.0 * (width*width + link2_length*link2_length)}" ixy="0.0" ixz="0.0" iyy="${mass / 12.0 * (link2_length*link2_length + width*width)}" iyz="0.0" izz="${mass / 12.0 * (width*width + width*width)}"/>
+      </inertial>
+    </link>
+    <!-- Joint 3: Prismatic -->
+    <joint name="${prefix}joint3" type="prismatic">
+      <limit effort="50" lower="0" upper="${link3_length - 2*axel_offset}" velocity="10"/>
+      <parent link="${prefix}link2"/>
+      <child link="${prefix}link3"/>
+      <origin xyz="0 ${width} ${link2_length - axel_offset*2}" rpy="0 1.5703 0"/>
+      <axis xyz="0 0 -1"/>
+      <dynamics damping="0.7"/>
+    </joint>
+    <!-- Link 3 -->
+    <link name="${prefix}link3">
+      <collision>
+        <origin xyz="0 0 ${link3_length/2 - axel_offset}" rpy="0 0 0"/>
+        <geometry>
+          <box size="${width} ${width} ${link3_length}"/>
+        </geometry>
+      </collision>
+      <visual>
+        <origin xyz="0 0 ${link3_length/2 - axel_offset}" rpy="0 0 0"/>
+        <geometry>
+          <box size="${width} ${width} ${link3_length}"/>
+        </geometry>
+        <material name="orange"/>
+      </visual>
+      <inertial>
+        <origin xyz="0 0 ${link3_length/2 - axel_offset}" rpy="0 0 0"/>
+        <mass value="${mass}"/>
+        <inertia ixx="${mass / 12.0 * (width*width + link3_length*link3_length)}" ixy="0.0" ixz="0.0" iyy="${mass / 12.0 * (link3_length*link3_length + width*width)}" iyz="0.0" izz="${mass / 12.0 * (width*width + width*width)}"/>
+      </inertial>
+    </link>
+    <!-- Tool Joint: Virtual -->
+    <joint name="${prefix}tool_joint" type="fixed">
+      <origin xyz="0 0 1" rpy="0 0 0" />
+      <parent link="${prefix}link3"/>
+      <child link="${prefix}tool_link" />
+    </joint>
+    <!-- Tool Link -->
+    <link name="${prefix}tool_link">
+    </link>
   </xacro:macro>
 </robot>
