Commit message: Correct the Frames and Joint positions as asked for

File: install/rrbot_description/share/rrbot_description/urdf/rrbot_description.urdf.xacro (robot description, xacro)
@@ -14,5 +14,5 @@
     <xacro:property name="link2_length" value="1" />
     <!-- Link 3 -->
-    <xacro:property name="link3_length" value="1" />
+    <xacro:property name="link3_length" value="1.2" />
     <!-- Link 4 -->
     <xacro:property name="camera_link" value="0.05" />
@@ -20,9 +20,12 @@
     <xacro:property name="axel_offset" value="0.05" />
     <!-- Space btw top of beam and the each joint -->
-    <!-- Joint 0: Fixed -->
-    <joint name="${prefix}base_joint" type="fixed">
+    <!-- Joint 1: Revolute -->
+    <joint name="${prefix}joint1" type="continuous">
       <xacro:insert_block name="origin" />
       <parent link="${parent}"/>
       <child link="${prefix}base_link" />
+      <origin xyz="0 0 0" rpy="0 0 0"/>
+      <axis xyz="0 0 1"/>
+      <dynamics damping="0.7"/>
     </joint>
     <!-- Base Link -->
@@ -47,16 +50,14 @@
       </inertial>
     </link>
-    <!-- Joint 1: Revolute -->
-    <joint name="${prefix}joint1" type="continuous">
+    <!-- Joint 1.5: Fixed -->
+    <joint name="${prefix}fixed_joint" type="fixed">
       <parent link="${prefix}base_link"/>
       <child link="${prefix}link1"/>
       <origin xyz="0 0 ${base_link_length}" rpy="0 0 0"/>
-      <axis xyz="0 0 1"/>
-      <dynamics damping="0.7"/>
     </joint>
     <!-- Link 1 -->
     <link name="${prefix}link1">
       <collision>
-        <origin xyz="0 0 ${link1_length/2 - axel_offset}" rpy="0 0 0"/>
+        <origin xyz="${link1_length/2 - axel_offset} 0 ${axel_offset}" rpy="0 1.5708 0"/>
         <geometry>
           <box size="${width} ${width} ${link1_length}"/>
@@ -64,5 +65,5 @@
       </collision>
       <visual>
-        <origin xyz="0 0 ${link1_length/2 - axel_offset}" rpy="0 0 0"/>
+        <origin xyz="${link1_length/2 - axel_offset} 0 ${axel_offset}" rpy="0 1.5708 0"/>
         <geometry>
           <box size="${width} ${width} ${link1_length}"/>
@@ -71,5 +72,5 @@
       </visual>
       <inertial>
-        <origin xyz="0 0 ${link1_length/2 - axel_offset}" rpy="0 0 0"/>
+        <origin xyz="${link1_length/2 - axel_offset} 0 ${axel_offset}" rpy="0 1.5708 0"/>
         <mass value="${mass}"/>
         <inertia ixx="${mass / 12.0 * (width*width + link1_length*link1_length)}" ixy="0.0" ixz="0.0" iyy="${mass / 12.0 * (link1_length*link1_length + width*width)}" iyz="0.0" izz="${mass / 12.0 * (width*width + width*width)}"/>
@@ -80,6 +81,6 @@
       <parent link="${prefix}link1"/>
       <child link="${prefix}link2"/>
-      <origin xyz="0 ${width} ${link1_length - axel_offset*2}" rpy="0 0 0"/>
-      <axis xyz="1 0 0"/>
+      <origin xyz="${link1_length - 2*axel_offset} 0 ${2*axel_offset}" rpy="0 0 0"/>
+      <axis xyz="0 0 1"/>
       <dynamics damping="0.7"/>
     </joint>
@@ -87,5 +88,5 @@
     <link name="${prefix}link2">
       <collision>
-        <origin xyz="0 0 ${link2_length/2 - axel_offset}" rpy="0 0 0"/>
+        <origin xyz="${link2_length/2 - axel_offset} 0 ${axel_offset}" rpy="0 1.5708 0"/>
         <geometry>
           <box size="${width} ${width} ${link2_length}"/>
@@ -93,5 +94,5 @@
       </collision>
       <visual>
-        <origin xyz="0 0 ${link2_length/2 - axel_offset}" rpy="0 0 0"/>
+        <origin xyz="${link2_length/2 - axel_offset} 0 ${axel_offset}" rpy="0 1.5708 0"/>
         <geometry>
           <box size="${width} ${width} ${link2_length}"/>
@@ -100,5 +101,5 @@
       </visual>
       <inertial>
-        <origin xyz="0 0 ${link2_length/2 - axel_offset}" rpy="0 0 0"/>
+        <origin xyz="${link2_length/2 - axel_offset} 0 ${axel_offset}" rpy="0 1.5708 0"/>
         <mass value="${mass}"/>
         <inertia ixx="${mass / 12.0 * (width*width + link2_length*link2_length)}" ixy="0.0" ixz="0.0" iyy="${mass / 12.0 * (link2_length*link2_length + width*width)}" iyz="0.0" izz="${mass / 12.0 * (width*width + width*width)}"/>
@@ -110,6 +111,6 @@
       <parent link="${prefix}link2"/>
       <child link="${prefix}link3"/>
-      <origin xyz="0 ${width} ${link2_length - axel_offset*2}" rpy="0 1.5703 0"/>
-      <axis xyz="0 0 -1"/>
+      <origin xyz="${link2_length - axel_offset} 0 ${axel_offset}" rpy="0 0 0"/>
+      <axis xyz="0 0 1"/>
       <dynamics damping="0.7"/>
     </joint>
@@ -117,5 +118,5 @@
     <link name="${prefix}link3">
       <collision>
-        <origin xyz="0 0 ${link3_length/2 - axel_offset}" rpy="0 0 0"/>
+        <origin xyz="${axel_offset} 0 ${-link3_length/2 + axel_offset}" rpy="0 0 0"/>
         <geometry>
           <box size="${width} ${width} ${link3_length}"/>
@@ -123,5 +124,5 @@
       </collision>
       <visual>
-        <origin xyz="0 0 ${link3_length/2 - axel_offset}" rpy="0 0 0"/>
+        <origin xyz="${axel_offset} 0 ${-link3_length/2 + axel_offset}" rpy="0 0 0"/>
         <geometry>
           <box size="${width} ${width} ${link3_length}"/>
@@ -130,5 +131,5 @@
       </visual>
       <inertial>
-        <origin xyz="0 0 ${link3_length/2 - axel_offset}" rpy="0 0 0"/>
+        <origin xyz="${axel_offset} 0 ${-link3_length/2 + axel_offset}" rpy="0 0 0"/>
         <mass value="${mass}"/>
         <inertia ixx="${mass / 12.0 * (width*width + link3_length*link3_length)}" ixy="0.0" ixz="0.0" iyy="${mass / 12.0 * (link3_length*link3_length + width*width)}" iyz="0.0" izz="${mass / 12.0 * (width*width + width*width)}"/>

File: src/rrbot_simulation_files/rrbot_description/urdf/rrbot_description.urdf.xacro (robot description, xacro)
@@ -14,5 +14,5 @@
     <xacro:property name="link2_length" value="1" />
     <!-- Link 3 -->
-    <xacro:property name="link3_length" value="1" />
+    <xacro:property name="link3_length" value="1.2" />
     <!-- Link 4 -->
     <xacro:property name="camera_link" value="0.05" />
@@ -20,9 +20,12 @@
     <xacro:property name="axel_offset" value="0.05" />
     <!-- Space btw top of beam and the each joint -->
-    <!-- Joint 0: Fixed -->
-    <joint name="${prefix}base_joint" type="fixed">
+    <!-- Joint 1: Revolute -->
+    <joint name="${prefix}joint1" type="continuous">
       <xacro:insert_block name="origin" />
       <parent link="${parent}"/>
       <child link="${prefix}base_link" />
+      <origin xyz="0 0 0" rpy="0 0 0"/>
+      <axis xyz="0 0 1"/>
+      <dynamics damping="0.7"/>
     </joint>
     <!-- Base Link -->
@@ -47,16 +50,14 @@
       </inertial>
     </link>
-    <!-- Joint 1: Revolute -->
-    <joint name="${prefix}joint1" type="continuous">
+    <!-- Joint 1.5: Fixed -->
+    <joint name="${prefix}fixed_joint" type="fixed">
       <parent link="${prefix}base_link"/>
       <child link="${prefix}link1"/>
-      <origin xyz="0 ${width} ${base_link_length - axel_offset}" rpy="0 1.5708 0"/>
-      <axis xyz="1 0 0"/>
-      <dynamics damping="0.7"/>
+      <origin xyz="0 0 ${base_link_length}" rpy="0 0 0"/>
     </joint>
     <!-- Link 1 -->
     <link name="${prefix}link1">
       <collision>
-        <origin xyz="0 0 ${link1_length/2 - axel_offset}" rpy="0 0 0"/>
+        <origin xyz="${link1_length/2 - axel_offset} 0 ${axel_offset}" rpy="0 1.5708 0"/>
         <geometry>
           <box size="${width} ${width} ${link1_length}"/>
@@ -64,5 +65,5 @@
       </collision>
       <visual>
-        <origin xyz="0 0 ${link1_length/2 - axel_offset}" rpy="0 0 0"/>
+        <origin xyz="${link1_length/2 - axel_offset} 0 ${axel_offset}" rpy="0 1.5708 0"/>
         <geometry>
           <box size="${width} ${width} ${link1_length}"/>
@@ -71,5 +72,5 @@
       </visual>
       <inertial>
-        <origin xyz="0 0 ${link1_length/2 - axel_offset}" rpy="0 0 0"/>
+        <origin xyz="${link1_length/2 - axel_offset} 0 ${axel_offset}" rpy="0 1.5708 0"/>
         <mass value="${mass}"/>
         <inertia ixx="${mass / 12.0 * (width*width + link1_length*link1_length)}" ixy="0.0" ixz="0.0" iyy="${mass / 12.0 * (link1_length*link1_length + width*width)}" iyz="0.0" izz="${mass / 12.0 * (width*width + width*width)}"/>
@@ -80,6 +81,6 @@
       <parent link="${prefix}link1"/>
       <child link="${prefix}link2"/>
-      <origin xyz="0 ${width} ${link1_length - axel_offset*2}" rpy="0 0 0"/>
-      <axis xyz="1 0 0"/>
+      <origin xyz="${link1_length - 2*axel_offset} 0 ${2*axel_offset}" rpy="0 0 0"/>
+      <axis xyz="0 0 1"/>
       <dynamics damping="0.7"/>
     </joint>
@@ -87,5 +88,5 @@
     <link name="${prefix}link2">
       <collision>
-        <origin xyz="0 0 ${link2_length/2 - axel_offset}" rpy="0 0 0"/>
+        <origin xyz="${link2_length/2 - axel_offset} 0 ${axel_offset}" rpy="0 1.5708 0"/>
         <geometry>
           <box size="${width} ${width} ${link2_length}"/>
@@ -93,5 +94,5 @@
       </collision>
       <visual>
-        <origin xyz="0 0 ${link2_length/2 - axel_offset}" rpy="0 0 0"/>
+        <origin xyz="${link2_length/2 - axel_offset} 0 ${axel_offset}" rpy="0 1.5708 0"/>
         <geometry>
           <box size="${width} ${width} ${link2_length}"/>
@@ -100,5 +101,5 @@
       </visual>
       <inertial>
-        <origin xyz="0 0 ${link2_length/2 - axel_offset}" rpy="0 0 0"/>
+        <origin xyz="${link2_length/2 - axel_offset} 0 ${axel_offset}" rpy="0 1.5708 0"/>
         <mass value="${mass}"/>
         <inertia ixx="${mass / 12.0 * (width*width + link2_length*link2_length)}" ixy="0.0" ixz="0.0" iyy="${mass / 12.0 * (link2_length*link2_length + width*width)}" iyz="0.0" izz="${mass / 12.0 * (width*width + width*width)}"/>
@@ -110,6 +111,6 @@
       <parent link="${prefix}link2"/>
       <child link="${prefix}link3"/>
-      <origin xyz="0 ${width} ${link2_length - axel_offset*2}" rpy="0 1.5703 0"/>
-      <axis xyz="0 0 -1"/>
+      <origin xyz="${link2_length - axel_offset} 0 ${axel_offset}" rpy="0 0 0"/>
+      <axis xyz="0 0 1"/>
       <dynamics damping="0.7"/>
     </joint>
@@ -117,5 +118,5 @@
     <link name="${prefix}link3">
       <collision>
-        <origin xyz="0 0 ${link3_length/2 - axel_offset}" rpy="0 0 0"/>
+        <origin xyz="${axel_offset} 0 ${-link3_length/2 + axel_offset}" rpy="0 0 0"/>
         <geometry>
           <box size="${width} ${width} ${link3_length}"/>
@@ -123,5 +124,5 @@
       </collision>
       <visual>
-        <origin xyz="0 0 ${link3_length/2 - axel_offset}" rpy="0 0 0"/>
+        <origin xyz="${axel_offset} 0 ${-link3_length/2 + axel_offset}" rpy="0 0 0"/>
         <geometry>
           <box size="${width} ${width} ${link3_length}"/>
@@ -130,5 +131,5 @@
       </visual>
       <inertial>
-        <origin xyz="0 0 ${link3_length/2 - axel_offset}" rpy="0 0 0"/>
+        <origin xyz="${axel_offset} 0 ${-link3_length/2 + axel_offset}" rpy="0 0 0"/>
         <mass value="${mass}"/>
         <inertia ixx="${mass / 12.0 * (width*width + link3_length*link3_length)}" ixy="0.0" ixz="0.0" iyy="${mass / 12.0 * (link3_length*link3_length + width*width)}" iyz="0.0" izz="${mass / 12.0 * (width*width + width*width)}"/>
