Commit message: Add the joint_controller.cpp in src/rrbot_gazebo/src and create a node with service

File: src/rrbot_simulation_files/rrbot_description/ros2_control/rrbot.ros2_control.xacro (robot description, xacro)
@@ -10,6 +10,6 @@
       </hardware> -->
       <hardware>
-          <plugin>gazebo_ros2_control/GazeboSystem</plugin>
-        </hardware>
+        <plugin>gazebo_ros2_control/GazeboSystem</plugin>
+      </hardware>
       <joint name="${prefix}joint1">
         <command_interface name="position">
@@ -46,4 +46,21 @@
         <state_interface name="effort"/>
       </joint>
+      <joint name="${prefix}joint3">
+        <command_interface name="position">
+          <param name="min">-10</param>
+          <param name="max">10</param>
+        </command_interface>
+        <command_interface name="velocity">
+          <param name="min">-10</param>
+          <param name="max">10</param>
+        </command_interface>
+        <command_interface name="effort">
+          <param name="min">-100</param>
+          <param name="max">100</param>
+        </command_interface>
+        <state_interface name="position"/>
+        <state_interface name="velocity"/>
+        <state_interface name="effort"/>
+      </joint>
     </ros2_control>
   </xacro:macro>
